File: PCB/Copy-Paste-Pad.kicad_pcb (KiCad board)
At the start: 2 copper layers, 65 x 80 mm, 18 parts, among them SW1 SW_Push_45deg, SW2 SW_Push_45deg, SW3 SW_Push_45deg, SW4 SW_Push_45deg, SW5 SW_Push_45deg, SW6 SW_Push_45deg, SW7 SW_Push_45deg, SW9 SW_Push_45deg, U1 MOUDLE-SEEEDUINO-XIAO, U3 ER_OLEDM0.91_1x-I2C

Commit message: small changes: PCB
fixing the 5v to 3v and wewirring everything to be more pretty
Parts:
- moved SW6 182.1 mm to (55.6, 43.2)
- moved D1 182.1 mm to (16.9, 18.3)
- moved D2 182.1 mm to (36.9, 18.3)
- moved D3 182.1 mm to (56.9, 18.3)
- moved D4 182.1 mm to (16.9, 38.3)
- moved D5 182.1 mm to (36.9, 38.3)
- moved D6 182.1 mm to (56.9, 38.3)
- moved D7 182.1 mm to (16.9, 58.3)
- moved D8 182.1 mm to (56.9, 58.3)
- moved SW1 182.1 mm to (15.6, 23.3)
- moved SW2 182.1 mm to (35.6, 23.2)
- moved SW3 182.1 mm to (55.6, 23.2)
- moved SW4 182.1 mm to (15.6, 43.2)
- moved SW5 182.1 mm to (35.6, 43.2)
- moved SW7 182.1 mm to (15.6, 63.2)
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Connections:
- U1 pad 12: unconnected-(U1-3V3-Pad12) -> Net-(U1-3V3)
- U1 pad 14: Net-(U1-5V) -> unconnected-(U1-5V-Pad14)
- U3 pad 2: Net-(U1-5V) -> Net-(U1-3V3)
Routing:
- net Net-(U1-3V3): track 0.00 -> 88.2 mm, vias 0 -> 2
- net Net-(U1-5V): track 82.6 -> 0.00 mm
- net Net-(U1-GND): track 71.8 -> 83.1 mm
- net Row 2: track 50.5 -> 44.4 mm
- net Row 0: track 96.3 -> 95.1 mm, vias 1 -> 4
- net Row 1: track 65.8 -> 66.8 mm, vias 1 -> 2
Other:
- outline, holes or cut-outs redrawn
