File: PCB/Copy-Paste-Pad.kicad_sch (KiCad schematic)
At the start: 18 parts, among them SW1 SW_Push_45deg, SW2 SW_Push_45deg, SW3 SW_Push_45deg, SW4 SW_Push_45deg, SW5 SW_Push_45deg, SW6 SW_Push_45deg, SW7 SW_Push_45deg, SW9 SW_Push_45deg, U1 MOUDLE-SEEEDUINO-XIAO, U3 ER_OLEDM0.91_1x-I2C

Commit message: small changes: PCB
fixing the 5v to 3v and wewirring everything to be more pretty
Connections:
- net at U1.12 (3V3): now also U3.2 (VCC)
- net at U1.14 (5V): no longer U3.2 (VCC)
Changed lines of the file:
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@@
-	(wire
-		(pts
-			(xy 101.6 45.72) (xy 101.6 54.61)
-		)
-		(stroke
-			(width 0)
-			(type default)
-		)
-	)
 	(wire
 		(pts
@@
 	(wire
 		(pts
+			(xy 101.6 50.8) (xy 101.6 54.61)
+		)
+		(stroke
+			(width 0)
+			(type default)
+		)
+	)
+	(wire
+		(pts
 			(xy 214.63 101.6) (xy 234.95 101.6)
 		)
@@
 	(wire
 		(pts
+			(xy 76.2 50.8) (xy 101.6 50.8)
+		)
+		(stroke
+			(width 0)
+			(type default)
+		)
+	)
+	(wire
+		(pts
 			(xy 234.95 78.74) (xy 247.65 78.74)
 		)
@@
 		)
 		(stroke
-			(width 0)
-			(type default)
-		)
-	)
-	(wire
-		(pts
-			(xy 76.2 45.72) (xy 101.6 45.72)
-		)
-		(stroke
